File: pcb-board/ddr_pcb/ddr_pcb.kicad_sch (KiCad schematic)
At the start: 1 part, among them U1 RP2040_Zero

Commit message: yay update
Parts:
- added D1, D2, D3, D4: LED, LED_THT:LED_D1.8mm_W1.8mm_H2.4mm_Horizontal_O1.27mm_Z1.6mm, symbol Device:LED
- added R1, R2, R3, R4: Resistor, Resistor_THT:R_Axial_DIN0207_L6.3mm_D2.5mm_P10.16mm_Horizontal, symbol ScottoKeebs:Placeholder_Resistor
- added S1, S2, S3, S4: Keyswitch, ScottoKeebs_Choc:Choc_V1, symbol ScottoKeebs:Placeholder_Keyswitch
Connections:
- net LEFT: now reaches U1.17 (26)
- net LEFT: now also D4.1 (K)
- net DOWN: now reaches U1.18 (27)
- net DOWN: now also D3.1 (K)
- net RIGHT: now reaches U1.19 (28)
- net RIGHT: now also D2.1 (K)
- net UP: now reaches U1.20 (29)
- net UP: now also D1.1 (K)
- net VCC: now reaches U1.23 (5V)
- net VCC: now also S1.1, S2.1, S3.1, S4.1
- new net: R2.2, S2.2
- new net: R3.2, S3.2
- new net: D3.2 (A), R3.1
- new net: D2.2 (A), R2.1
- new net: D1.2 (A), R1.1
- new net: R1.2, S1.2
- new net: D4.2 (A), R4.1
- new net: R4.2, S4.2
Other:
- moved on the sheet: U1

Commit message: like my 3rd pcb design
Parts:
- S1, S2, S3, S4: footprint ScottoKeebs_Choc:Choc_V1 -> ScottoKeebs_Choc:Choc_20x20mm
Connections:
- net DOWN: now also S3.1; no longer D3.1 (K)
- net LEFT: now also S4.1; no longer D4.1 (K)
- net RIGHT: now also S2.1; no longer D2.1 (K)
- net UP: now also S1.1; no longer D1.1 (K)
- net GND: now reaches U1.22 (GND)
- net GND: now also D1.1 (K), D2.1 (K), D3.1 (K), D4.1 (K)
- removed net VCC: S1.1, S2.1, S3.1, S4.1, U1.23 (5V)
Changed lines of the file:
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@@
 	(wire
 		(pts
-			(xy 199.39 85.09) (xy 199.39 88.9)
+			(xy 199.39 82.55) (xy 199.39 88.9)
 		)
 		(stroke
@@
 	(wire
 		(pts
-			(xy 190.5 100.33) (xy 194.31 100.33)
+			(xy 199.39 57.15) (xy 199.39 63.5)
 		)
 		(stroke
@@
 	(wire
 		(pts
-			(xy 212.09 101.6) (xy 214.63 101.6)
+			(xy 177.8 82.55) (xy 177.8 87.63)
 		)
 		(stroke
@@
 	(wire
 		(pts
-			(xy 199.39 59.69) (xy 199.39 63.5)
+			(xy 177.8 57.15) (xy 177.8 63.5)
 		)
 		(stroke
@@
 		)
 	)
-	(wire
-		(pts
-			(xy 212.09 76.2) (xy 214.63 76.2)
-		)
-		(stroke
-			(width 0)
-			(type default)
-		)
-	)
-	(wire
-		(pts
-			(xy 190.5 76.2) (xy 194.31 76.2)
-		)
-		(stroke
-			(width 0)
-			(type default)
-		)
-	)
-	(wire
-		(pts
-			(xy 177.8 83.82) (xy 177.8 87.63)
-		)
-		(stroke
-			(width 0)
-			(type default)
-		)
-	)
-	(wire
-		(pts
-			(xy 177.8 59.69) (xy 177.8 63.5)
-		)
-		(stroke
-			(width 0)
-			(type default)
-		)
-	)
 	(global_label "RIGHT"
 		(shape input)
-		(at 214.63 76.2 0)
+		(at 199.39 57.15 90)
 		(fields_autoplaced yes)
 		(effects
@@
 		)
 		(property "Intersheetrefs" "${INTERSHEET_REFS}"
-			(at 223.0581 76.2 0)
+			(at 199.39 48.7219 90)
 			(effects
 				(font
@@
 		)
 	)
-	(global_label "VCC"
-		(shape input)
-		(at 199.39 59.69 90)
+	(global_label "GND"
+		(shape input)
+		(at 190.5 100.33 0)
 		(fields_autoplaced yes)
 		(effects
@@
 		)
 		(property "Intersheetrefs" "${INTERSHEET_REFS}"
-			(at 199.39 53.0762 90)
+			(at 197.3557 100.33 0)
 			(effects
 				(font
@@
 		)
 	)
-	(global_label "VCC"
-		(shape input)
-		(at 177.8 59.69 90)
+	(global_label "RIGHT"
+		(shape input)
+		(at 129.54 76.2 180)
+		(fields_autoplaced yes)
+		(effects
+			(font
+				(size 1.27 1.27)
+			)
+			(justify right)
+		)
+		(property "Intersheetrefs" "${INTERSHEET_REFS}"
+			(at 121.1119 76.2 0)
+			(effects
+				(font
+					(size 1.27 1.27)
+				)
+				(justify right)
+				(hide yes)
+			)
+		)
+	)
+	(global_label "GND"
+		(shape input)
+		(at 212.09 76.2 0)
 		(fields_autoplaced yes)
 		(effects
@@
 		)
 		(property "Intersheetrefs" "${INTERSHEET_REFS}"
-			(at 177.8 53.0762 90)
+			(at 218.9457 76.2 0)
 			(effects
 				(font
@@
 		)
 	)
-	(global_label "RIGHT"
-		(shape input)
-		(at 129.54 76.2 180)
+	(global_label "GND"
+		(shape input)
+		(at 212.09 101.6 0)
+		(fields_autoplaced yes)
+		(effects
+			(font
+				(size 1.27 1.27)
+			)
+			(justify left)
+		)
+		(property "Intersheetrefs" "${INTERSHEET_REFS}"
+			(at 218.9457 101.6 0)
+			(effects
+				(font
+					(size 1.27 1.27)
+				)
+				(justify left)
+				(hide yes)
+			)
+		)
+	)
+	(global_label "DOWN"
+		(shape input)
+		(at 177.8 82.55 90)
+		(fields_autoplaced yes)
+		(effects
+			(font
+				(size 1.27 1.27)
+			)
+			(justify left)
+		)
+		(property "Intersheetrefs" "${INTERSHEET_REFS}"
+			(at 177.8 74.1824 90)
+			(effects
+				(font
+					(size 1.27 1.27)
+				)
+				(justify left)
+				(hide yes)
+			)
+		)
+	)
+	(global_label "DOWN"
+		(shape input)
+		(at 129.54 78.74 180)
 		(fields_autoplaced yes)
 		(effects
@@
 		)
 		(property "Intersheetrefs" "${INTERSHEET_REFS}"
-			(at 121.1119 76.2 0)
-			(effects
-				(font
-					(size 1.27 1.27)
-				)
-				(justify right)
-				(hide yes)
-			)
-		)
-	)
-	(global_label "VCC"
-		(shape input)
-		(at 199.39 85.09 90)
+			(at 121.1724 78.74 0)
+			(effects
+				(font
+					(size 1.27 1.27)
+				)
+				(justify right)
+				(hide yes)
+			)
+		)
+	)
+	(global_label "GND"
+		(shape input)
+		(at 129.54 68.58 180)
+		(fields_autoplaced yes)
+		(effects
+			(font
+				(size 1.27 1.27)
+			)
+			(justify right)
+		)
+		(property "Intersheetrefs" "${INTERSHEET_REFS}"
+			(at 122.6843 68.58 0)
+			(effects
+				(font
+					(size 1.27 1.27)
+				)
+				(justify right)
+				(hide yes)
+			)
+		)
+	)
+	(global_label "GND"
+		(shape input)
+		(at 190.5 76.2 0)
 		(fields_autoplaced yes)
 		(effects
@@
 		)
 		(property "Intersheetrefs" "${INTERSHEET_REFS}"
-			(at 199.39 78.4762 90)
+			(at 197.3557 76.2 0)
 			(effects
 				(font
@@
 		)
 	)
-	(global_label "DOWN"
-		(shape input)
-		(at 194.31 100.33 0)
+	(global_label "LEFT"
+		(shape input)
+		(at 199.39 82.55 90)
 		(fields_autoplaced yes)
 		(effects
@@
 		)
 		(property "Intersheetrefs" "${INTERSHEET_REFS}"
-			(at 202.6776 100.33 0)
+			(at 199.39 75.3315 90)
 			(effects
 				(font
@@
 		)
 	)
-	(global_label "VCC"
-		(shape input)
-		(at 177.8 83.82 90)
+	(global_label "UP"
+		(shape input)
+		(at 177.8 57.15 90)
 		(fields_autoplaced yes)
 		(effects
@@
 		)
 		(property "Intersheetrefs" "${INTERSHEET_REFS}"
-			(at 177.8 77.2062 90)
-			(effects
-				(font
-					(size 1.27 1.27)
-				)
-				(justify left)
-				(hide yes)
-			)
-		)
-	)
-	(global_label "DOWN"
-		(shape input)
-		(at 129.54 78.74 180)
-		(fields_autoplaced yes)
-		(effects
-			(font
-				(size 1.27 1.27)
-			)
-			(justify right)
-		)
-		(property "Intersheetrefs" "${INTERSHEET_REFS}"
-			(at 121.1724 78.74 0)
-			(effects
-				(font
-					(size 1.27 1.27)
-				)
-				(justify right)
-				(hide yes)
-			)
-		)
-	)
-	(global_label "VCC"
-		(shape input)
-		(at 129.54 66.04 180)
-		(fields_autoplaced yes)
-		(effects
-			(font
-				(size 1.27 1.27)
-			)
-			(justify right)
-		)
-		(property "Intersheetrefs" "${INTERSHEET_REFS}"
-			(at 122.9262 66.04 0)
-			(effects
-				(font
-					(size 1.27 1.27)
-				)
-				(justify right)
-				(hide yes)
-			)
-		)
-	)
-	(global_label "LEFT"
-		(shape input)
-		(at 214.63 101.6 0)
-		(fields_autoplaced yes)
-		(effects
-			(font
-				(size 1.27 1.27)
-			)
-			(justify left)
-		)
-		(property "Intersheetrefs" "${INTERSHEET_REFS}"
-			(at 221.8485 101.6 0)
-			(effects
-				(font
-					(size 1.27 1.27)
-				)
-				(justify left)
-				(hide yes)
-			)
-		)
-	)
-	(global_label "UP"
-		(shape input)
-		(at 194.31 76.2 0)
-		(fields_autoplaced yes)
-		(effects
-			(font
-				(size 1.27 1.27)
-			)
-			(justify left)
-		)
-		(property "Intersheetrefs" "${INTERSHEET_REFS}"
-			(at 199.8957 76.2 0)
+			(at 177.8 51.5643 90)
 			(effects
 				(font
@@
 			)
 		)
-		(property "Footprint" "ScottoKeebs_Choc:Choc_V1"
+		(property "Footprint" "ScottoKeebs_Choc:Choc_20x20mm"
 			(at 201.93 66.04 0)
 			(effects
@@
 			)
 		)
-		(property "Footprint" "ScottoKeebs_Choc:Choc_V1"
+		(property "Footprint" "ScottoKeebs_Choc:Choc_20x20mm"
 			(at 180.34 90.17 0)
 			(effects
@@
 			)
 		)
-		(property "Footprint" "ScottoKeebs_Choc:Choc_V1"
+		(property "Footprint" "ScottoKeebs_Choc:Choc_20x20mm"
 			(at 180.34 66.04 0)
 			(effects
@@
 			)
 		)
-		(property "Footprint" "ScottoKeebs_Choc:Choc_V1"
+		(property "Footprint" "ScottoKeebs_Choc:Choc_20x20mm"
 			(at 201.93 91.44 0)
 			(effects
